Commit message: Adding base_link origin to mesh

File: vilma_vehicle_description/urdf/vehicle.xacro (robot description, xacro)
@@ -6,8 +6,12 @@
   <link name="base_link">
     <visual>
-      <origin xyz="${vehicle_info['/**']['ros__parameters']['wheel_base']/2.0 + 0.77} 0 -${vehicle_info['/**']['ros__parameters']['wheel_radius']/2.0}" rpy="${pi/2.0} 0 ${pi}"/>
+      <origin xyz="0 0 0" rpy="${pi/2.0} 0 ${pi}"/>
+      <geometry>
+        <mesh filename="package://vilma_vehicle_description/mesh/punto/model_base_link_origin.dae" scale="0.7133 0.7133 0.7133"/>
+      </geometry>
+      <!-- <origin xyz="${vehicle_info['/**']['ros__parameters']['wheel_base']/2.0 + 0.77} 0 -${vehicle_info['/**']['ros__parameters']['wheel_radius']/2.0}" rpy="${pi/2.0} 0 ${pi}"/>
       <geometry>
         <mesh filename="package://vilma_vehicle_description/mesh/punto/model.dae" scale="1 1 1"/>
-      </geometry>
+      </geometry> -->
     </visual>
   </link>

Commit message: Updating launch and mesh position

File: vilma_vehicle_description/urdf/vehicle.xacro (robot description, xacro)
@@ -6,5 +6,5 @@
   <link name="base_link">
     <visual>
-      <origin xyz="0 0 0" rpy="${pi/2.0} 0 ${pi}"/>
+      <origin xyz="${vehicle_info['/**']['ros__parameters']['wheel_base']/2.0} 0 0" rpy="${pi/2.0} 0 ${pi}"/>
       <geometry>
         <mesh filename="package://vilma_vehicle_description/mesh/punto/model_base_link_origin.dae" scale="0.7133 0.7133 0.7133"/>

Commit message: Setting mesh position

File: vilma_vehicle_description/urdf/vehicle.xacro (robot description, xacro)
@@ -6,5 +6,5 @@
   <link name="base_link">
     <visual>
-      <origin xyz="${vehicle_info['/**']['ros__parameters']['wheel_base']/2.0} 0 0" rpy="${pi/2.0} 0 ${pi}"/>
+      <origin xyz="0 0 ${vehicle_info['/**']['ros__parameters']['wheel_radius']}" rpy="${pi/2.0} 0 ${pi}"/>
       <geometry>
         <mesh filename="package://vilma_vehicle_description/mesh/punto/model_base_link_origin.dae" scale="0.7133 0.7133 0.7133"/>
